File: hardware/jellybean/jellybean.sch (KiCad schematic (older format))
At the start: 92 parts

Commit message: I2S header
Parts:
- added D?: USBLED, symbol LED
- added P?: I2S, symbol CONN_5X2
- added R?: 470, symbol R
Connections:
- net GND: now also D?.2 (K), P?.10, P?.2, P?.4, P?.6, P?.8
- net VCC: now also P?.1
- net I2S0_TX_SCK: now reaches U?.112 (P3_0)
- net I2S0_TX_SCK: now also P?.7
- net I2S0_TX_WS: now reaches U?.114 (P3_1)
- net I2S0_TX_WS: now also P?.5
- net I2S0_TX_SDA: now reaches U?.116 (P3_2)
- net I2S0_TX_SDA: now also P?.3
- net USB0_IND0: now reaches U?.95 (P2_6)
- net USB0_IND0: now also R?.1
- net I2S0_TX_MCLK: now reaches U?.99 (CLK2)
- net I2S0_TX_MCLK: now also P?.9
- new net: D?.1 (A), R?.2
- no-connect marks 34 -> 30
Other:
- moved on the sheet: R?

Commit message: indicator LEDs
Parts:
- added D?: LED3, symbol LED
- added D?: VCCLED, symbol LED
- added D?: LED2, symbol LED
- added D?: 1V8LED, symbol LED
- added D?: LED1, symbol LED
- added R? (x5): 470, symbol R
Connections:
- net EN1V8: now also R?.1
- net GND: now also D?.2 (K), D?.2 (K), D?.2 (K), D?.2 (K), D?.2 (K)
- net VCC: now also R?.1
- new net: D?.1 (A), R?.2 (x5)
- new net LED1: R?.1
- new net LED2: R?.1
- new net LED3: R?.1
Other:
- moved on the sheet: D?, K?, P?

Commit message: VBUS voltage divider per errata sheet
Parts:
- added R?: 15k, symbol R
- added R?: 33k, symbol R
Connections:
- net GND: now also R?.2
- net VBUS: now also R?.1; no longer U?.21 (USB0_VBUS)
- new net: R?.1, R?.2, U?.21 (USB0_VBUS)
Changed lines of the file:
@@
-EESchema Schematic File Version 2  date Mon Apr  9 23:21:54 2012
+EESchema Schematic File Version 2  date Mon Apr  9 23:27:28 2012
 LIBS:power
 LIBS:device
@@
 Comment4 ""
 $EndDescr
-Text Label 3150 6650 3    40   ~ 0
-LED3
-Text Label 2850 6650 3    40   ~ 0
-LED2
-Text Label 2550 6650 3    40   ~ 0
-LED1
+Wire Wire Line
+	4300 5000 3500 5000
+Wire Wire Line
+	3500 5000 3500 4450
+Connection ~ 3000 4450
+Wire Wire Line
+	3500 4450 3000 4450
+Wire Wire Line
+	3000 4550 3000 4350
 Wire Wire Line
 	3750 7400 3750 7500
@@
 	1600 3000 1700 3000
 Wire Wire Line
-	2900 3550 2900 4900
+	3700 3550 3700 4900
 Wire Wire Line
 	750  8400 1050 8400
@@
 Connection ~ 13800 2650
 Wire Wire Line
-	13700 2650 14300 2650
+	14300 2650 13700 2650
 Connection ~ 13800 650
 Wire Wire Line
-	13700 650  14300 650
+	14300 650  13700 650
 Wire Wire Line
 	13800 2650 13800 1850
@@
 Connection ~ 2500 3750
 Wire Wire Line
-	2900 3550 1100 3550
+	3700 3550 1100 3550
 Wire Wire Line
 	2500 3850 2500 3750
@@
 	1200 3250 1100 3250
 Wire Wire Line
-	4300 5000 3000 5000
-Wire Wire Line
-	4300 4700 2800 4700
+	4300 4700 3600 4700
 Wire Wire Line
 	7650 2050 7650 1950
@@
 Connection ~ 2300 5700
 Wire Wire Line
-	1850 5700 4300 5700
+	4300 5700 1850 5700
 Connection ~ 2500 5600
 Wire Wire Line
@@
 Connection ~ 1350 9350
 Wire Wire Line
-	1250 9350 1450 9350
+	1450 9350 1250 9350
 Connection ~ 950  9550
 Wire Wire Line
-	850  9550 1450 9550
+	1450 9550 850  9550
 Wire Wire Line
 	750  9750 750  9650
@@
 Connection ~ 10850 4600
 Wire Wire Line
-	11050 4600 9700 4600
+	9700 4600 11050 4600
 Connection ~ 10350 4200
 Wire Wire Line
-	10500 4200 9700 4200
+	9700 4200 10500 4200
 Connection ~ 2100 6000
 Wire Wire Line
@@
 	10350 4100 10350 4200
 Wire Wire Line
-	11050 4500 9700 4500
+	9700 4500 11050 4500
 Connection ~ 10650 4500
 Wire Wire Line
@@
 	950  9750 950  9550
 Wire Wire Line
-	650  9650 1450 9650
+	1450 9650 650  9650
 Connection ~ 750  9650
 Wire Wire Line
-	1050 9450 1450 9450
+	1450 9450 1050 9450
 Connection ~ 1150 9450
 Wire Wire Line
@@
 	11950 4200 12050 4200
 Wire Wire Line
-	6850 1300 6850 2050
+	6850 2050 6850 1300
 Wire Wire Line
 	11950 3900 12050 3900
@@
 	5650 2050 5650 1750
 Wire Wire Line
-	2900 4900 4300 4900
+	3700 4900 4300 4900
 Wire Wire Line
-	4300 5100 3100 5100
+	4300 5100 3800 5100
 Wire Wire Line
-	3100 5100 3100 3350
+	3800 5100 3800 3350
 Wire Wire Line
-	3100 3350 1100 3350
+	3800 3350 1100 3350
 Wire Wire Line
 	2500 4350 2500 4250
@@
 	2200 3750 2200 3850
 Wire Wire Line
-	1100 3450 2800 3450
+	1100 3450 3600 3450
 Wire Wire Line
 	11600 7850 11400 7850
@@
 	13300 4200 13050 4200
 Wire Wire Line
-	13900 1650 13350 1650
+	13350 1650 13900 1650
 Wire Wire Line
 	13550 2250 13550 2150
@@
 	15300 1850 15300 1950
 Wire Wire Line
-	14800 650  15900 650
+	15900 650  14800 650
 Connection ~ 15300 650
 Wire Wire Line
 	15500 1250 15500 1150
 Wire Wire Line
-	15900 2650 14800 2650
+	14800 2650 15900 2650
 Connection ~ 15300 2650
 Connection ~ 15500 2650
@@
 	15500 2050 15500 2150
 Wire Wire Line
-	12700 1550 13900 1550
+	13900 1550 12700 1550
 Wire Wire Line
-	12800 1450 12800 1650
+	12800 1650 12800 1450
 Wire Wire Line
 	12800 850  12800 950
 Wire Wire Line
-	15200 1550 16400 1550
+	16400 1550 15200 1550
 Connection ~ 16150 1550
 Wire Wire Line
@@
 	9600 1650 9900 1650
 Wire Wire Line
-	11100 1850 11100 1350
+	11100 1350 11100 1850
 Connection ~ 11100 1450
 Wire Wire Line
@@
 Connection ~ 6650 1400
 Wire Wire Line
-	6650 1300 6650 2050
+	6650 2050 6650 1300
 Wire Wire Line
 	15800 9450 16000 9450
@@
 	4800 9300 4800 9200
 Wire Wire Line
-	4700 8700 5050 8700
+	5050 8700 4700 8700
 Wire Wire Line
 	4300 8700 3900 8700
@@
 	4300 5800 4000 5800
 Wire Wire Line
-	2800 3450 2800 4700
+	3600 3450 3600 4700
 Wire Wire Line
 	3000 3750 2100 3750
@@
 Wire Wire Line
 	2800 3000 3000 3000
-Wire Wire Line
-	3000 3000 3000 5000
 Connection ~ 3000 3750
 Wire Wire Line
@@
 Wire Wire Line
 	3450 7400 3450 7500
+Wire Wire Line
+	3000 5150 3000 5050
+Wire Wire Line
+	3000 3000 3000 3850
+$Comp
+L GND #PWR?
+U 1 1 4F83C49F
+P 3000 5150
+F 0 "#PWR?" H 3000 5150 30  0001 C CNN
+F 1 "GND" H 3000 5080 30  0001 C CNN
+	1    3000 5150
+	1    0    0    -1
+$EndComp
+$Comp
+L R R?
+U 1 1 4F83C495
+P 3000 4800
+F 0 "R?" V 3080 4800 50  0000 C CNN
+F 1 "33k" V 3000 4800 50  0000 C CNN
+	1    3000 4800
+	1    0    0    -1
+$EndComp
+$Comp
+L R R?
+U 1 1 4F83C48F
+P 3000 4100
+F 0 "R?" V 3080 4100 50  0000 C CNN
+F 1 "15k" V 3000 4100 50  0000 C CNN
+	1    3000 4100
+	1    0    0    -1
+$EndComp
+Text Label 3150 6650 3    40   ~ 0
+LED3
+Text Label 2850 6650 3    40   ~ 0
+LED2
+Text Label 2550 6650 3    40   ~ 0
+LED1
 $Comp
 L VCC #PWR?
@@
 Text Label 4000 5100 0    40   ~ 0
 ID
-Text Label 4000 5000 0    40   ~ 0
+Text Label 2250 3750 0    40   ~ 0
 VBUS
 Text Label 4000 4900 0    40   ~ 0

Commit message: annotation
Parts:
- gave numbers to parts that had none: 107
Connections:
- net LED1: now also U2.3 (P4_1)
- net LED2: now also U2.8 (P4_2)
- net LED3: now also U2.14 (P4_7)
- no-connect marks 30 -> 27

Commit message: cosmetic cleanup
Connections:
- net VCCIO2: no longer C32.1, C33.1
- new net: C32.1, C33.1
Other:
- moved on the sheet: C22, C23, C25, C26, C29, C32, C33, C6, C8, FB1, J1, K1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

Commit message: some BOM details
Parts:
- FB1: Description (none) -> FERRITE CHIP 220 OHM 1400MA 0603; Manufacturer (none) -> Murata; Part Number (none) -> BLM18PG221SN1D
- U1: Description (none) -> IC USB DUAL ESD PROTECT 6TSOP; Manufacturer (none) -> NXP; Part Number (none) -> IP4220CZ6,125
- U2: Description (none) -> IC MCU 32BIT 144LQFP; Manufacturer (none) -> NXP; Part Number (none) -> LPC4330FBD144,551
- U3: Description (none) -> IC FLASH 8MBIT 8SOIC; Manufacturer (none) -> Winbond; Part Number (none) -> W25Q80BVSSIG
- U4: Description (none) -> IC CR-II CPLD 64MCELL 100-VQFP; Manufacturer (none) -> Xilinx; Part Number (none) -> XC2C64A-7VQG100C
- U5: Description (none) -> IC BUCK SYNC DUAL ADJ 0.8A 10SON; Manufacturer (none) -> Texas Instruments; Part Number (none) -> TPS62410
Changed lines of the file:
@@
-EESchema Schematic File Version 2  date Mon Apr  9 23:43:44 2012
+EESchema Schematic File Version 2  date Tue Apr 10 08:30:53 2012
 LIBS:power
 LIBS:device
@@
 F 0 "U2" H 7000 4900 60  0000 C CNN
 F 1 "LPC43XXFBD144" H 7000 4600 60  0000 C CNN
+F 4 "NXP" H 7000 4750 60  0001 C CNN "Manufacturer"
+F 5 "LPC4330FBD144,551" H 7000 4750 60  0001 C CNN "Part Number"
+F 6 "IC MCU 32BIT 144LQFP" H 7000 4750 60  0001 C CNN "Description"
 	1    7000 4750
 	1    0    0    -1
@@
 F 0 "U3" H 10450 1350 60  0000 C CNN
 F 1 "W25Q80BV" H 10450 1850 60  0000 C CNN
+F 4 "Winbond" H 10450 1600 60  0001 C CNN "Manufacturer"
+F 5 "W25Q80BVSSIG" H 10450 1600 60  0001 C CNN "Part Number"
+F 6 "IC FLASH 8MBIT 8SOIC" H 10450 1600 60  0001 C CNN "Description"
 	1    10450 1600
 	1    0    0    -1
@@
 F 0 "U5" H 14550 1600 60  0000 C CNN
 F 1 "TPS62410" H 14550 1950 60  0000 C CNN
+F 4 "Texas Instruments" H 14550 1650 60  0001 C CNN "Manufacturer"
+F 5 "TPS62410" H 14550 1650 60  0001 C CNN "Part Number"
+F 6 "IC BUCK SYNC DUAL ADJ 0.8A 10SON" H 14550 1650 60  0001 C CNN "Description"
 	1    14550 1650
 	1    0    0    -1
@@
 F 0 "U4" H 13600 7050 60  0000 C CNN
 F 1 "GSG-XC2C64A-7VQG100C" H 13600 6850 60  0000 C CNN
+F 4 "Xilinx" H 13600 6950 60  0001 C CNN "Manufacturer"
+F 5 "XC2C64A-7VQG100C" H 13600 6950 60  0001 C CNN "Part Number"
+F 6 "IC CR-II CPLD 64MCELL 100-VQFP" H 13600 6950 60  0001 C CNN "Description"
 	1    13600 6950
 	1    0    0    -1
@@
 F 0 "FB1" H 1950 3900 60  0000 C CNN
 F 1 "FILTER" H 1950 3650 60  0000 C CNN
+F 4 "Murata" H 1950 3750 60  0001 C CNN "Manufacturer"
+F 5 "BLM18PG221SN1D" H 1950 3750 60  0001 C CNN "Part Number"
+F 6 "FERRITE CHIP 220 OHM 1400MA 0603" H 1950 3750 60  0001 C CNN "Description"
 	1    1950 3750
 	1    0    0    -1
@@
 F 0 "U1" H 2450 3250 60  0000 C CNN
 F 1 "GSG-IP4220CZ6" H 2450 2750 60  0000 C CNN
+F 4 "NXP" H 2450 3000 60  0001 C CNN "Manufacturer"
+F 5 "IP4220CZ6,125" H 2450 3000 60  0001 C CNN "Part Number"
+F 6 "IC USB DUAL ESD PROTECT 6TSOP" H 2450 3000 60  0001 C CNN "Description"
 	1    2450 3000
 	1    0    0    -1

Commit message: fixed some things Jared noticed
Parts:
- removed P3: LPC_AUX, symbol CONN_16X2
- removed P4: BOOT_CTRL, symbol CONN_4X2
- added D7: USBLED0, symbol LED
- added P19: BOOT1, symbol CONN_3
- added P20: BOOT2, symbol CONN_3
- added P21: BOOT3, symbol CONN_3
- added P3: CONN_12X2, symbol CONN_12X2
- added P4: BOOT0, symbol CONN_3
- added R41, R42, R43: 10k, symbol R
- D6: value USBLED -> USBLED1
- FB1: Description FERRITE CHIP 220 OHM 1400MA 0603 -> FERRITE CHIP 220 OHM 2000MA 0805; Part Number BLM18PG221SN1D -> BLM21PG221SN1D
- K1: value BANK2_PWR -> BANK1_PWR
- R1, R2: value 10k -> 0
- R3: value 10k -> 470
Connections:
- net CTIN_7 is gone; now on net INTR: U2.97 (P6_9)
- net CTOUT_6 is gone; now on net CPLD_TDI: U2.82 (P6_5)
- net CTOUT_7 is gone; now on net LED3: U2.103 (P6_12)
- net BOOT0: now also R4.1; no longer R1.1
- net BOOT1: now also R41.1; no longer R2.1
- net BOOT2: now also R42.1; no longer R3.1
- net BOOT3: now also R43.1; no longer R4.1
- net CPLD_TCK: now also U2.74 (P6_1); no longer U2.73 (P6_0)
- net CPLD_TDI: no longer U2.78 (P6_2)
- net CPLD_TMS: now also U2.78 (P6_2); no longer U2.74 (P6_1)
- net CTIN_2: now also P3.9 (P9)
- net CTIN_4: now also P3.1 (P1)
- net CTIN_6: now also P3.15 (P15)
- net CTOUT_2: now also P3.7 (P7)
- net CTOUT_4: now also P3.3 (P3)
- net CTOUT_5: now also P3.5 (P5)
- net DBGEN: now also P3.21 (P21)
- net DM: now also R2.1; no longer J1.2 (D-), U1.1 (ESD1)
- net DP: now also R1.1; no longer J1.3 (D+), U1.3 (ESD2)
- net GND: now also D7.2 (K), P19.1 (P1), P20.1 (P1), P21.1 (P1), P3.10 (P10), P3.12 (P12), P3.14 (P14), P3.16 (P16), P3.18 (P18), P3.2 (P2), P3.20 (P20), P3.22 (P22), P3.24 (P24), P3.4 (P4), P3.6 (P6), P3.8 (P8), P4.1 (P1); no longer R1.2, R2.2, R3.2, R4.2
- net INTR: no longer U2.86 (P6_8)
- net LED3: no longer U2.14 (P4_7)
- net OEB: now also U2.95 (P2_6); no longer U2.85 (P6_7)
- net TRACECLK: now also P3.17 (P17)
- net TRST: now also P3.23 (P23)
- net U3_RXD: now also P3.11 (P11)
- net U3_TXD: now also P3.13 (P13)
- net USB0_IND0: now also R3.1, U2.86 (P6_8); no longer R29.1, U2.95 (P2_6)
- net VCC: now also U4.88 (VCCIO2), U4.98 (VCCIO2), P19.3 (P3), P20.3 (P3), P21.3 (P3), P4.3 (P3); no longer U4.38 (VCCIO1), U4.51 (VCCIO1)
- net VCCIO2: no longer K1.2 (PM), U4.88 (VCCIO2), U4.98 (VCCIO2)
- net WAKEUP: now also P3.19 (P19)
- removed net ID: J1.4 (ID), U1.4 (ESD3), U2.22 (USB0_ID)
- net SSP0_MISO renamed SPIFI_MISO
- net SSP0_MOSI renamed SPIFI_MOSI
- net SSP0_SCK renamed SPIFI_SCK
- net SSP0_SSEL renamed SPIFI_CS
- new net: J1.2 (D-), R2.2, U1.1 (ESD1)
- new net: J1.3 (D+), R1.2, U1.3 (ESD2)
- new net: P4.2 (PM), R4.2
- new net: P19.2 (PM), R41.2
- new net: P21.2 (PM), R43.2
- new net: P20.2 (PM), R42.2
- new net: D7.1 (A), R3.2
- new net USB0_IND1: R29.1, U2.85 (P6_7)
- new net VCCIO1: K1.2 (PM), U4.38 (VCCIO1), U4.51 (VCCIO1)
- no-connect marks 27 -> 32
Other:
- note added: "bank 1 power selection"
- note removed: "bank 2 power selection"
- moved on the sheet: D6, R29
