File: hardware/lollipop/lollipop.sch (KiCad schematic (older format))
At the start: 85 parts

Commit message: added some notes
Other:
- note added: "RX bandpass path"
- note added: "RX highpass path"
- note added: "RX lowpass path"
- note added: "TX bandpass path"
- note added: "TX highpass path"
- note added: "TX lowpass path"
- note added: "antenna diversity switches"
- note added: "balun here will not be needed when a\nboard is made with a direct connection\nto the MAX2837"
Changed lines of the file:
@@
-EESchema Schematic File Version 2  date Wed May  9 01:09:11 2012
+EESchema Schematic File Version 2  date Wed May  9 12:01:23 2012
 LIBS:power
 LIBS:device
@@
 Comment4 ""
 $EndDescr
+Text Notes 14800 9200 0    40   ~ 0
+balun here will not be needed when a\nboard is made with a direct connection\nto the MAX2837
+Text Notes 14800 2350 0    40   ~ 0
+balun here will not be needed when a\nboard is made with a direct connection\nto the MAX2837
+Text Notes 7250 7450 2    40   ~ 0
+RX bandpass path
+Text Notes 7250 6350 2    40   ~ 0
+RX lowpass path
+Text Notes 7250 5250 2    40   ~ 0
+RX highpass path
+Text Notes 7250 4050 2    40   ~ 0
+TX highpass path
+Text Notes 7250 2950 2    40   ~ 0
+TX lowpass path
+Text Notes 7250 1850 2    40   ~ 0
+TX bandpass path
 Wire Wire Line
 	4500 1650 4250 1650
@@
 Connection ~ 1150 4750
 Connection ~ 1150 6150
+Text Notes 3350 3850 2    40   ~ 0
+antenna diversity switches
 Text Label 4250 1650 0    40   ~ 0
 SWTXV1

Commit message: adjusted blocking cap values for low frequency response
Parts:
- removed C? (x13): 100pF, symbol C
- removed C? (x2): 47pF, symbol C
- added C? (x14): 2.2nF, symbol C
- C?: value 100pF -> 2.2nF
Connections:
- net at U?.1 (RFC): now also C?.2
- net at U?.5 (RF2): now also C?.1
- net at T?.3 (PR1): now also C?.2 (x2)
- net at T?.4 (PR2): now also C?.2 (x2)
- net at U?.2 (OUT): now also C?.1
- net at U?.1 (RFC): now also C?.1
- net at U?.5 (RF2): now also C?.2
- net at P?.1 (RF): now also C?.2
- net at U?.2 (OUT): now also C?.2
- net at U?.17 (MIX1_OPN): now also C?.2
- net at U?.18 (MIX1_OPP): now also C?.2
- net at U?.23 (MIX2_IPP): now also C?.2
- net at U?.24 (MIX2_IPN): now also C?.2
- net at U?.1 (OUT1): now also C?.1 (x2)
- net at U?.5 (INPUT): now also C?.1 (x5)
- net at U?.3 (OUT2): now also C?.1 (x4)
- net at U?.1 (OUT1): now also C?.2 (x2)

Commit message: mixer output inductors for power, todo list
Parts:
- added L? (x4): INDUCTOR, symbol INDUCTOR
Connections:
- net VCC: now also L?.1, L?.1, L?.2, L?.2
- net at C?.2, U?.17 (MIX1_OPN): now also L?.2
- net at C?.2, U?.18 (MIX1_OPP): now also L?.2
- net at C?.1, U?.27 (MIX2_OPN): now also L?.1
- net at C?.1, U?.28 (MIX2_OPP): now also L?.1
Other:
- note added: "TO DO:\nmixer output inductor values\ncheck balun pinouts\nswitch control logic\ncontrol header\npower in header\nclock in header\nimpedance matching\namplification\nmisc. mixer connections"
