File: hardware/hackrf-one/frontend.sch (KiCad schematic (older format))
At the start: 144 parts, among them J10 GND_CLIP, J2 RF-SHIELD-FRAME, J3 RF-SHIELD-COVER, J4 MOUNTING_HOLE, J5 MOUNTING_HOLE, J6 MOUNTING_HOLE, J7 MOUNTING_HOLE, J8 MOUNTING_HOLE, J9 MOUNTING_HOLE, P13 GPO1, P17 GPO6, P19 GPO3, P21 REF_IN, P27 MIXER_SDATA, P31 MIXER_SCLK, P32 MIXER_ENX, P33 MIXER_RESETX, P34 MIX_BYPASS, P35 !MIX_BYPASS, P4 ANTENNA, P42 TX, P43 RX, P44 HP, P45 LP, P46 TX_MIX_BP, P47 RX_MIX_BP, P48 TX_AMP, P49 RX_AMP, P50 AMP_BYPASS, P51 !TX_AMP_PWR, P52 !RX_AMP_PWR, P6 GPO4, P7 GPO2, Q1 MOSFET_P, Q2 MOSFET_P, Q4 MOSFET_P, T1 MIX_IN_BALUN, T2 MIX_OUT_BALUN, U1 SKY13350, U10 SKY13350, U11 SKY13350, U12 SKY13317, U13 MGA-81563, U14 SKY13317, U2 SKY13350, U25 MGA-81563, U3 RX_LOWPASS_FILTER, U4 RFFC5072, U5 SKY13350, U6 SKY13350, U7 SKY13350, U8 RX_HIGHPASS_FILTER, U9 SKY13317

Commit message: Kicad parts remapping
Parts:
- C1, C10, C11, C12, C13, C14, C15, C16, C160, C161, C162, C163, C166, C17, C171, C18, C19, C2, C20, C21, C22, C23, C24, C25, C26, C27, C28, C29, C3, C30, C31, C32, C33, C34, C35, C36, C37, C38, C39, C4, C40, C41, C42, C43, C44, C45, C46, C47, C48, C49, C5, C50, C51, C52, C53, C54, C55, C56, C57, C58, C59, C6, C60, C61, C62, C63, C64, C65, C66, C67, C7, C70, C8, C9: symbol C -> Device:C
- D1: symbol GSG-DIODE-TVS-BI -> hackrf:GSG-DIODE-TVS-BI
- J10, J4, J5, J6, J7, J8, J9, P13, P17, P19, P21, P27, P31, P32, P33, P34, P35, P42, P43, P44, P45, P46, P47, P48, P49, P50, P51, P52, P6, P7: symbol CONN_1 -> hackrf-one-rescue:CONN_1
- J2: symbol RF-SHIELD-FRAME -> hackrf:RF-SHIELD-FRAME
- J3: symbol RF-SHIELD-COVER -> hackrf:RF-SHIELD-COVER
- L1, L12, L13, L2, L3, L4, L5: symbol INDUCTOR -> hackrf-one-rescue:INDUCTOR
- P4: symbol GSG-RF-CONN -> hackrf:GSG-RF-CONN
- Q1, Q2, Q4: symbol MOSFET_P -> hackrf-one-rescue:MOSFET_P
- R1, R2, R24, R29, R3, R36, R4, R5, R6: symbol R -> Device:R
- T1, T2: symbol BALUN-B0310J50100AHF -> hackrf:BALUN-B0310J50100AHF
- U1, U10, U11, U2, U5, U6, U7: symbol SKY13350 -> hackrf:SKY13350
- U12, U14, U9: symbol SKY13317 -> hackrf:SKY13317
- U13, U25: symbol MGA-81563 -> hackrf:MGA-81563
- U3: symbol FIL-LP0603 -> hackrf:FIL-LP0603
- U4: symbol RFFC5072 -> hackrf:RFFC5072
- U8: symbol FIL-DEA -> hackrf:FIL-DEA
Connections:
- wire segments 367 -> 438

Commit message: Added protection diodes and related components to schematic. Related (but not the diodes) added to the PCB
Parts:
- removed D1: GSG-DIODE-TVS-BI, hackrf:GSG-0402, symbol hackrf:GSG-DIODE-TVS-BI
- added C117, C172: 100nF, hackrf:GSG-0402, symbol Device:C
- added D10, D11, D12: SMP1330, symbol hackrf:D_Limiter
- added R38, R39, R40: 10k, hackrf:GSG-0402, symbol Device:R
Connections:
- wire segments 438 -> 448
Other:
- moved on the sheet: C58, C63

Commit message: Improved Bias T design to use two inductors
Parts:
- added C173: 1pF, hackrf:GSG-0402, symbol Device:C
- added L14: 3.3uH, hackrf:GSG-0603, symbol hackrf-one-rescue:INDUCTOR
- added R42, R43, R44: 1.5k, hackrf:GSG-0402, symbol Device:R
- D10, D11, D12: footprint (none) -> gsg-modules:SMP1330-085LF; Part Number SKY1330-085LF -> SMP1330-085LF
- L13: value 10uH -> 0.56uH; Description INDUCTR 10UH 220MA 20% 0603 SMD -> INDUCTOR 560nH ±5% 70mA 8.1Ω 0603; Manufacturer Taiyo Yuden -> Sunlord; Part Number BRL1608T100M -> SDWL1608CR56JSTF
- R38, R39, R40: Description RES 22K OHM 1/10W 5% 0402 SMD -> RES 10K OHM 1/16W 5% 0402 SMD; Manufacturer Panasonic -> Stackpole; Part Number ERJ-2GEJ223X -> RMCF0402JT10K0
Connections:
- wire segments 448 -> 461
Other:
- moved on the sheet: C171, C63, L13, Q4, R36

Commit message: Updated U13 and U25 Rx and Tx amps from MGA-81563 to TRF37B73
Parts:
- removed U13, U25: MGA-81563, hackrf:GSG-SOT363, symbol hackrf:MGA-81563
- added U13, U25: TRF37B73, Package_SON:WSON-8-1EP_2x2mm_P0.5mm_EP0.9x1.6mm, symbol hackrf:TRF37B73
Connections:
- wire segments 461 -> 456
Other:
- moved on the sheet: C117, C160, C161, C162, C163, C50, C52, C53, C55, C57, C58, C59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

Commit message: Updated U1, 2, 5, 6, 10, 11 from SKY13350 to SKY13453
Parts:
- removed C11, C19: 33pF, hackrf:GSG-0402, symbol Device:C
- removed U1, U10, U11, U2, U5, U6, U7: SKY13350, hackrf:GSG-SKY13350-385LF, symbol hackrf:SKY13350
- added U1, U10, U11, U2, U5, U6, U7: SKY13453, gsg-modules:SKY13453-385LF, symbol hackrf:SKY13453
Connections:
- wire segments 456 -> 449
Other:
- moved on the sheet: C30

Commit message: Made SMP1330 a 3-terminal device to match the data sheet
Parts:
- removed P42: TX, hackrf:GSG-TESTPOINT-50MIL, symbol hackrf-one-rescue:CONN_1
- D10, D11, D12: symbol hackrf:D_Limiter -> hackrf:D_Limiter_DualAn
Connections:
- net GND: now also D10.2 (K), D12.1 (A1), D12.3 (A2); no longer D10.1 (K), D12.2 (A)
- net RX_AMP_IN: now also D10.1 (A1); no longer C58.1, D10.2 (A)
- net VAA: now also D11.2 (K); no longer D11.1 (K)
- new net: C64.2, D11.1 (A1), R39.1
- new net: C58.1, D10.3 (A2)
- new net: C172.1, D11.3 (A2), D12.2 (K), R40.2
Other:
- moved on the sheet: C172, R40

Commit message: Moved -rescue lib symbols to hackrf.lib
Parts:
- J10, J4, J5, J6, J7, J8, J9, P13, P17, P19, P21, P27, P31, P32, P33, P34, P35, P43, P44, P45, P46, P47, P48, P49, P50, P51, P52, P6, P7: symbol hackrf-one-rescue:CONN_1 -> hackrf:CONN_1
- L1, L12, L13, L14, L2, L3, L4, L5: symbol hackrf-one-rescue:INDUCTOR -> hackrf:INDUCTOR
- Q1, Q2, Q4: symbol hackrf-one-rescue:MOSFET_P -> hackrf:MOSFET_P
Changed lines of the file:
@@
 $EndComp
 $Comp
-L hackrf-one-rescue:INDUCTOR L12
+L hackrf:INDUCTOR L12
 U 1 1 503BF2DC
 P 14350 5950
@@
 $EndComp
 $Comp
-L hackrf-one-rescue:MOSFET_P Q2
+L hackrf:MOSFET_P Q2
 U 1 1 503BF2D7
 P 12400 5850
@@
 $EndComp
 $Comp
-L hackrf-one-rescue:INDUCTOR L3
+L hackrf:INDUCTOR L3
 U 1 1 503BF2B7
 P 4800 5050
@@
 $EndComp
 $Comp
-L hackrf-one-rescue:INDUCTOR L2
+L hackrf:INDUCTOR L2
 U 1 1 503BF2A7
 P 4800 4750
@@
 $EndComp
 $Comp
-L hackrf-one-rescue:MOSFET_P Q1
+L hackrf:MOSFET_P Q1
 U 1 1 502E69D1
 P 10200 8500
@@
 $EndComp
 $Comp
-L hackrf-one-rescue:INDUCTOR L5
+L hackrf:INDUCTOR L5
 U 1 1 502C6D12
 P 8950 9300
@@
 $EndComp
 $Comp
-L hackrf-one-rescue:INDUCTOR L4
+L hackrf:INDUCTOR L4
 U 1 1 4FB55E30
 P 5300 5550
@@
 $EndComp
 $Comp
-L hackrf-one-rescue:INDUCTOR L1
+L hackrf:INDUCTOR L1
 U 1 1 502AFA8C
 P 3900 3750
@@
 	1600 2150 1600 2250
 $Comp
-L hackrf-one-rescue:CONN_1 P6
+L hackrf:CONN_1 P6
 U 1 1 526B7056
 P 5100 4500
@@
 $EndComp
 $Comp
-L hackrf-one-rescue:CONN_1 P19
+L hackrf:CONN_1 P19
 U 1 1 5280432B
 P 5000 4500
@@
 	5000 4250 5000 4350
 $Comp
-L hackrf-one-rescue:CONN_1 P7
+L hackrf:CONN_1 P7
 U 1 1 528044D2
 P 4750 1850
@@
 $EndComp
 $Comp
-L hackrf-one-rescue:CONN_1 P13
+L hackrf:CONN_1 P13
 U 1 1 528044D9
 P 4750 1750
@@
 $EndComp
 $Comp
-L hackrf-one-rescue:CONN_1 P21
+L hackrf:CONN_1 P21
 U 1 1 528044E0
 P 6700 9550
@@
 	5700 1950 5700 1850
 $Comp
-L hackrf-one-rescue:CONN_1 P17
+L hackrf:CONN_1 P17
 U 1 1 52805038
 P 5700 1700
@@
 MIXER_SDATA
 $Comp
-L hackrf-one-rescue:CONN_1 P27
+L hackrf:CONN_1 P27
 U 1 1 528054F2
 P 3450 8600
@@
 $EndComp
 $Comp
-L hackrf-one-rescue:CONN_1 P31
+L hackrf:CONN_1 P31
 U 1 1 528054F9
 P 3450 8700
@@
 $EndComp
 $Comp
-L hackrf-one-rescue:CONN_1 P32
+L hackrf:CONN_1 P32
 U 1 1 52805500
 P 3450 8800
@@
 $EndComp
 $Comp
-L hackrf-one-rescue:CONN_1 P33
+L hackrf:CONN_1 P33
 U 1 1 52805507
 P 3450 8900
@@
 !TX_AMP_PWR
 $Comp
-L hackrf-one-rescue:CONN_1 P34
+L hackrf:CONN_1 P34
 U 1 1 52805C27
 P 3450 9000
@@
 $EndComp
 $Comp
-L hackrf-one-rescue:CONN_1 P35
+L hackrf:CONN_1 P35
 U 1 1 52805C2E
 P 3450 9100
@@
 $EndComp
 $Comp
-L hackrf-one-rescue:CONN_1 P43
+L hackrf:CONN_1 P43
 U 1 1 52805C3C
 P 3450 9300
@@
 	3600 9000 3700 9000
 $Comp
-L hackrf-one-rescue:CONN_1 P44
+L hackrf:CONN_1 P44
 U 1 1 52805C47
 P 3450 9400
@@
 $EndComp
 $Comp
-L hackrf-one-rescue:CONN_1 P45
+L hackrf:CONN_1 P45
 U 1 1 52805C4E
 P 3450 9500
@@
 $EndComp
 $Comp
-L hackrf-one-rescue:CONN_1 P46
+L hackrf:CONN_1 P46
 U 1 1 52805C55
 P 3450 9600
@@
 $EndComp
 $Comp
-L hackrf-one-rescue:CONN_1 P47
+L hackrf:CONN_1 P47
 U 1 1 52805C5C
 P 3450 9700
@@
 	3600 9400 3700 9400
 $Comp
-L hackrf-one-rescue:CONN_1 P48
+L hackrf:CONN_1 P48
 U 1 1 52805C67
 P 3450 9800
@@
 $EndComp
 $Comp
-L hackrf-one-rescue:CONN_1 P49
+L hackrf:CONN_1 P49
 U 1 1 52805C6E
 P 3450 9900
@@
 $EndComp
 $Comp
-L hackrf-one-rescue:CONN_1 P50
+L hackrf:CONN_1 P50
 U 1 1 52805C75
 P 3450 10000
@@
 $EndComp
 $Comp
-L hackrf-one-rescue:CONN_1 P51
+L hackrf:CONN_1 P51
 U 1 1 52805C7C
 P 3450 10100
@@
 	3600 9800 3700 9800
 $Comp
-L hackrf-one-rescue:CONN_1 P52
+L hackrf:CONN_1 P52
 U 1 1 52805C87
 P 3450 10200
@@
 $EndComp
 $Comp
-L hackrf-one-rescue:CONN_1 J4
+L hackrf:CONN_1 J4
 U 1 1 528FA040
 P 850 9850
@@
 	850  10000 850  10100
 $Comp
-L hackrf-one-rescue:CONN_1 J5
+L hackrf:CONN_1 J5
 U 1 1 528FA22A
 P 1050 9850
@@
 	1050 10000 1050 10100
 $Comp
-L hackrf-one-rescue:CONN_1 J6
+L hackrf:CONN_1 J6
 U 1 1 528FA29A
 P 1250 9850
@@
 	1250 10000 1250 10100
 $Comp
-L hackrf-one-rescue:CONN_1 J7
+L hackrf:CONN_1 J7
 U 1 1 528FA2A8
 P 1450 9850
@@
 	1450 10000 1450 10100
 $Comp
-L hackrf-one-rescue:CONN_1 J8
+L hackrf:CONN_1 J8
 U 1 1 528FA2B6
 P 1650 9850
@@
 	1650 10000 1650 10100
 $Comp
-L hackrf-one-rescue:CONN_1 J9
+L hackrf:CONN_1 J9
 U 1 1 528FA2C4
 P 1850 9850
@@
 $EndComp
 $Comp
-L hackrf-one-rescue:CONN_1 J10
+L hackrf:CONN_1 J10
 U 1 1 5293FD15
 P 2600 9850
@@
 $EndComp
 $Comp
-L hackrf-one-rescue:INDUCTOR L13
+L hackrf:INDUCTOR L13
 U 1 1 52EA1189
 P 15550 7650
@@
 $EndComp
 $Comp
-L hackrf-one-rescue:MOSFET_P Q4
+L hackrf:MOSFET_P Q4
 U 1 1 52EA11B0
 P 15450 6300
@@
 	16200 7700 16200 7750
 $Comp
-L hackrf-one-rescue:INDUCTOR L?
+L hackrf:INDUCTOR L?
 U 1 1 5F078049
 P 15550 6950
