File: hardware/hackrf-one/mcu.kicad_sch (KiCad schematic)
At the start: 131 parts, among them J1 USB-MICRO-B, P20 GPIO, P22 I2S, P23 DBGEN, P24 TRST, P25 LPC_ISP, P26 LPC_JTAG, P28 SD, P29 CPLD_JTAG, P3 GND, P30 BANK2_AUX, P5 LEDS, P68 SPIFI_CS, P69 VREGMODE, P70 EN_1V8, P71 ID, P73 P1_2, P74 P1_1, P75 GP_CLKIN, P76 GP_CLKIN, P77 GP_CLKIN, P78 GP_CLKIN, P79 GP_CLKIN, P80 SHIELD, P81 SPIFI_SIO2, P82 SPIFI_SIO3, Q5 MOSFET_P, SW1 DFU, SW2 RESET, U15 TVS, U20 W25Q80, U21 TPS62410, U23 LPC4320FBD144, U24 GSG-XC2C64A-7VQG100C, X2 MCU_XTAL, X3 RTC_XTAL

Commit message: HackRF One: update 100 nF capacitor part selection
Parts:
- C128, C129, C130, C131, C132, C133, C134, C135, C136, C137, C138, C139, C140, C141, C142, C144, C147, C148, C149, C150, C151, C152, C153, C154: Manufacturer Murata -> Samsung; Part Number GRM155R61A104KA01D -> CL05A104KA5NNNC
